File: Esquemático_KiCad/untitled.kicad_sch (KiCad schematic)
At the start: 76 parts, among them J1 AUDIO_IN, J2 Conn_01x02, U15 OPA1679, U3 OPA1679, U4 OPA1679, U8 OPA1679

Commit message: Commit Ficheiros Atualizados, PSpice e kiCad
Parts:
- R20, R7: value 6.4k -> 10k
- R21, R8: value 50.8k -> 45.97k
- R22, R9: value 50.8k -> 10k
Changed lines of the file:
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@@
 			)
 		)
-		(property "Value" "50.8k"
+		(property "Value" "10k"
 			(at 68.326 38.862 90)
 			(effects
@@
 			)
 		)
-		(property "Value" "50.8k"
+		(property "Value" "10k"
 			(at 67.056 88.392 90)
 			(effects
@@
 			)
 		)
-		(property "Value" "50.8k"
+		(property "Value" "45.97k"
 			(at 68.58 24.13 90)
 			(effects
@@
 			)
 		)
-		(property "Value" "50.8k"
+		(property "Value" "45.97k"
 			(at 67.31 73.66 90)
 			(effects
@@
 			)
 		)
-		(property "Value" "6.4k"
+		(property "Value" "10k"
 			(at 41.91 50.7999 0)
 			(effects
@@
 			)
 		)
-		(property "Value" "6.4k"
+		(property "Value" "10k"
 			(at 40.64 100.3299 0)
 			(effects
